Commit message: picture

File: d2c_robot_description/urdf/d2c_robot_description.urdf (robot description, URDF)
Before this commit: robot d2c_description, 5 links, 4 joints
Links:
- link base_link: mass 0.068503 -> 0.087818
- link link3: mass 0.081122 -> 0.073185
- link link4: mass 0.0095064 -> 0.05126
Joints:
- joint joint1: origin xyz=-0.00056185 0.0125 0.0429 rpy=0 0 0 -> xyz=-0.016486 -0.0032999 0.0429 rpy=0 0 0
- joint joint2: axis 1 0 0 -> -1 0 0; origin xyz=-0.0254 0.0125 0.02335 rpy=0 0 0 -> xyz=0.0254 -0.0125 0.02335 rpy=0 0 0
- joint joint3: axis -1 0 0 -> 1 0 0; origin xyz=-0.036 -0.03025 0.18425 rpy=0 0 0 -> xyz=0.036 0.03025 0.18425 rpy=0 0 0
- joint joint4: axis 1 0 0 -> -1 0 -0.0013953; origin xyz=0.037937 -0.184 -9.3958E-05 rpy=0 0 0 -> xyz=-0.0429 0.17 -6E-05 rpy=0 0 0

Commit message: get object data setup

File: d2c_robot_description/urdf/d2c_robot_description.urdf (robot description, URDF)
Before this commit: robot d2c_robot_description, 5 links, 4 joints
Joints:
- joint joint1: axis 0 0 -1 -> 0 0 1
- joint joint2: axis -1 0 0 -> 1 0 0
